Commit message: Updated URDF to separate end effector from wrist

File: src/tomato_description/urdf/tomato_arm.urdf.xacro (robot description, xacro)
@@ -89,3 +89,17 @@
         </visual>
     </link>
+    <joint name="joint_5" type="fixed">
+        <parent link="wrist_link"/>
+        <child link="end_effector_link"/>
+        <origin xyz="0.0345 0 0" rpy="0 0 0"/>
+    </joint>
+    <link name="end_effector_link">
+        <visual>
+            <origin xyz="-0.3647 0 -0.10597" rpy="0 0 0"/>
+            <geometry>
+                <mesh filename="package://tomato_description/meshes/end_effector_link.stl"/>
+            </geometry>
+            <material name="color5"/>
+        </visual>
+    </link>
 </robot>

Commit message: IK kinda working

File: src/tomato_description/urdf/tomato_arm.urdf.xacro (robot description, xacro)
@@ -103,3 +103,9 @@
         </visual>
     </link>
+    <link name="tool_tip_link"/>
+    <joint name="tool_tip_joint" type="fixed">
+        <parent link="end_effector_link"/>
+        <child link="tool_tip_link"/>
+        <origin xyz="0.03193 0 0" rpy="0 0 0"/>
+    </joint>
 </robot>

Commit message: Added new end effector mesh

File: src/tomato_description/urdf/tomato_arm.urdf.xacro (robot description, xacro)
@@ -28,5 +28,5 @@
         <parent link="base_link"/>
         <child link="shoulder_link"/>
-        <origin xyz="0 0 0" rpy="0 0 0"/>
+        <origin xyz="0 0 0" rpy="0 0 1.5708"/>
         <axis xyz="0 0 1"/>
         <limit effort="1.0" velocity="2.0"/>
@@ -98,5 +98,7 @@
             <origin xyz="-0.3647 0 -0.10597" rpy="0 0 0"/>
             <geometry>
-                <mesh filename="package://tomato_description/meshes/end_effector_link.stl"/>
+                <mesh
+                    filename="package://tomato_description/meshes/end_effector_link.stl"
+                    scale="0.001 0.001 0.001"/>
             </geometry>
             <material name="color5"/>
@@ -107,5 +109,5 @@
         <parent link="end_effector_link"/>
         <child link="tool_tip_link"/>
-        <origin xyz="0.03193 0 0" rpy="0 0 0"/>
+        <origin xyz="0.124 0 0.04416" rpy="0 0 0"/>
     </joint>
 </robot>

Commit message: URDF w camera mount

File: src/tomato_description/urdf/tomato_arm.urdf.xacro (robot description, xacro)
@@ -1,4 +1,26 @@
 <?xml version="1.0"?>
 <robot xmlns:xacro="http://www.ros.org/wiki/xacro" name="tomato_arm">
+    <!-- ===================================================== -->
+    <!-- CAMERA PARAMETERS                                     -->
+    <!-- ===================================================== -->
+    <!--
+        base_link convention:
+        +X = forward
+        -X = backward
+        +Y = robot-left
+        -Y = robot-right
+        +Z = upward
+    -->
+    <!-- Both camera lens centers are 20 cm behind the shoulder -->
+    <xacro:property name="camera_x" value="-0.20"/>
+    <!-- Camera lens centers are 65 cm above base_link -->
+    <xacro:property name="camera_height" value="0.65"/>
+    <!-- 41 degrees downward -->
+    <xacro:property name="camera_pitch" value="0.715585"/>
+    <!-- Distance between the two camera lens centers -->
+    <xacro:property name="camera_baseline" value="0.10"/>
+    <!-- ===================================================== -->
+    <!-- MATERIALS                                             -->
+    <!-- ===================================================== -->
     <material name="color1">
         <color rgba="1.0 0.0 0.0 1.0"/>
@@ -16,9 +38,18 @@
         <color rgba="0.65 0.20 0.85 1.0"/>
     </material>
+    <!-- ===================================================== -->
+    <!-- ROBOT ARM                                             -->
+    <!-- ===================================================== -->
     <link name="base_link">
         <visual>
-            <origin xyz="0 0 0" rpy="0 0 0"/>
-            <geometry>
-            <mesh filename="package://tomato_description/meshes/base_link.stl"/>
+            <!--
+                Rotate only the base STL by 90 degrees.
+                This does not rotate base_link, the arm,
+                the camera transforms, or the IK coordinate frame.
+            -->
+            <origin xyz="0 0 0" rpy="0 0 1.5708"/>
+            <geometry>
+                <mesh
+                    filename="package://tomato_description/meshes/base_link.stl"/>
             </geometry>
             <material name="color1"/>
@@ -28,5 +59,6 @@
         <parent link="base_link"/>
         <child link="shoulder_link"/>
-        <origin xyz="0 0 0" rpy="0 0 1.5708"/>
+        <!-- Arm orientation already matches the real robot -->
+        <origin xyz="0 0 0" rpy="0 0 0"/>
         <axis xyz="0 0 1"/>
         <limit effort="1.0" velocity="2.0"/>
@@ -36,5 +68,6 @@
             <origin xyz="0 0 0" rpy="0 0 0"/>
             <geometry>
-                <mesh filename="package://tomato_description/meshes/shoulder_link.stl"/>
+                <mesh
+                    filename="package://tomato_description/meshes/shoulder_link.stl"/>
             </geometry>
             <material name="color2"/>
@@ -46,5 +79,9 @@
         <origin xyz="0 0 0.10597" rpy="0 -1.5708 0"/>
         <axis xyz="0 1 0"/>
-        <limit lower="-1.618" upper="1.595" effort="1.0" velocity="2.0"/>
+        <limit
+            lower="-1.618"
+            upper="1.595"
+            effort="1.0"
+            velocity="2.0"/>
     </joint>
     <link name="forearm_link">
@@ -52,5 +89,6 @@
             <origin xyz="0 0 -0.10597" rpy="0 0 0"/>
             <geometry>
-                <mesh filename="package://tomato_description/meshes/forearm_link.stl"/>
+                <mesh
+                    filename="package://tomato_description/meshes/forearm_link.stl"/>
             </geometry>
             <material name="color3"/>
@@ -62,5 +100,9 @@
         <origin xyz="0.1778 0 0" rpy="0 0 0"/>
         <axis xyz="0 1 0"/>
-        <limit lower="-1.825" upper="1.792" effort="1.0" velocity="2.0"/>
+        <limit
+            lower="-1.825"
+            upper="1.792"
+            effort="1.0"
+            velocity="2.0"/>
     </joint>
     <link name="elbow_link">
@@ -68,5 +110,6 @@
             <origin xyz="-0.1778 0 -0.10597" rpy="0 0 0"/>
             <geometry>
-                <mesh filename="package://tomato_description/meshes/elbow_link.stl"/>
+                <mesh
+                    filename="package://tomato_description/meshes/elbow_link.stl"/>
             </geometry>
             <material name="color4"/>
@@ -78,5 +121,9 @@
         <origin xyz="0.1524 0 0" rpy="0 0 0"/>
         <axis xyz="0 1 0"/>
-        <limit lower="-1.855" upper="1.786" effort="1.0" velocity="2.0"/>
+        <limit
+            lower="-1.855"
+            upper="1.786"
+            effort="1.0"
+            velocity="2.0"/>
     </joint>
     <link name="wrist_link">
@@ -84,5 +131,6 @@
             <origin xyz="-0.3302 0 -0.10597" rpy="0 0 0"/>
             <geometry>
-                <mesh filename="package://tomato_description/meshes/wrist_link.stl"/>
+                <mesh
+                    filename="package://tomato_description/meshes/wrist_link.stl"/>
             </geometry>
             <material name="color5"/>
@@ -111,3 +159,121 @@
         <origin xyz="0.124 0 0.04416" rpy="0 0 0"/>
     </joint>
+    <!-- ===================================================== -->
+    <!-- CAMERA STAND                                          -->
+    <!-- ===================================================== -->
+    <link name="camera_stand_link">
+        <visual>
+            <!--
+                The camera_stand_link frame is at its bottom.
+                The box is centered so it extends from z=0 to z=0.65.
+            -->
+            <origin
+                xyz="0 0 ${camera_height / 2.0}"
+                rpy="0 0 0"/>
+            <geometry>
+                <box size="0.03 0.03 ${camera_height}"/>
+            </geometry>
+            <material name="color3"/>
+        </visual>
+    </link>
+    <joint name="camera_stand_joint" type="fixed">
+        <parent link="base_link"/>
+        <child link="camera_stand_link"/>
+        <!-- Stand is 20 cm behind the shoulder along -X -->
+        <origin
+            xyz="${camera_x} 0 0"
+            rpy="0 0 0"/>
+    </joint>
+    <!-- ===================================================== -->
+    <!-- CAMERA MOUNT                                          -->
+    <!-- ===================================================== -->
+    <link name="camera_mount_link">
+        <visual>
+            <origin xyz="0 0 0" rpy="0 0 0"/>
+            <geometry>
+                <!-- Crossbar extends left/right along Y -->
+                <box size="0.04 0.16 0.03"/>
+            </geometry>
+            <material name="color4"/>
+        </visual>
+    </link>
+    <joint name="camera_mount_joint" type="fixed">
+        <parent link="camera_stand_link"/>
+        <child link="camera_mount_link"/>
+        <!--
+            No forward position offset.
+            The lens centers remain at x = -0.20 m.
+            Positive pitch rotates local +X toward:
+              +X forward
+              -Z downward
+        -->
+        <origin
+            xyz="0 0 ${camera_height}"
+            rpy="0 ${camera_pitch} 0"/>
+    </joint>
+    <!-- ===================================================== -->
+    <!-- LEFT CAMERA                                           -->
+    <!-- ===================================================== -->
+    <link name="left_camera_link">
+        <visual>
+            <origin xyz="0 0 0" rpy="0 0 0"/>
+            <geometry>
+                <box size="0.035 0.025 0.025"/>
+            </geometry>
+            <material name="color1"/>
+        </visual>
+    </link>
+    <joint name="left_camera_joint" type="fixed">
+        <parent link="camera_mount_link"/>
+        <child link="left_camera_link"/>
+        <!-- Left camera is at Y = +5 cm -->
+        <origin
+            xyz="0 ${camera_baseline / 2.0} 0"
+            rpy="0 0 0"/>
+    </joint>
+    <!-- ===================================================== -->
+    <!-- RIGHT CAMERA                                          -->
+    <!-- ===================================================== -->
+    <link name="right_camera_link">
+        <visual>
+            <origin xyz="0 0 0" rpy="0 0 0"/>
+            <geometry>
+                <box size="0.035 0.025 0.025"/>
+            </geometry>
+            <material name="color1"/>
+        </visual>
+    </link>
+    <joint name="right_camera_joint" type="fixed">
+        <parent link="camera_mount_link"/>
+        <child link="right_camera_link"/>
+        <!-- Right camera is at Y = -5 cm -->
+        <origin
+            xyz="0 ${-camera_baseline / 2.0} 0"
+            rpy="0 0 0"/>
+    </joint>
+    <!-- ===================================================== -->
+    <!-- CAMERA OPTICAL FRAMES                                 -->
+    <!-- ===================================================== -->
+    <link name="left_camera_optical_frame"/>
+    <joint name="left_camera_optical_joint" type="fixed">
+        <parent link="left_camera_link"/>
+        <child link="left_camera_optical_frame"/>
+        <!--
+            ROS optical convention:
+            +Z = viewing direction
+            +X = image right
+            +Y = image down
+        -->
+        <origin
+            xyz="0 0 0"
+            rpy="-1.5708 0 -1.5708"/>
+    </joint>
+    <link name="right_camera_optical_frame"/>
+    <joint name="right_camera_optical_joint" type="fixed">
+        <parent link="right_camera_link"/>
+        <child link="right_camera_optical_frame"/>
+        <origin
+            xyz="0 0 0"
+            rpy="-1.5708 0 -1.5708"/>
+    </joint>
 </robot>

Commit message: New stereo calibration

File: src/tomato_description/urdf/tomato_arm.urdf.xacro (robot description, xacro)
@@ -16,8 +16,22 @@
     <!-- Camera lens centers are 65 cm above base_link -->
     <xacro:property name="camera_height" value="0.65"/>
-    <!-- 41 degrees downward -->
-    <xacro:property name="camera_pitch" value="0.715585"/>
+    <!-- 35 degrees downward -->
+    <xacro:property name="camera_pitch" value="0.610865"/>
     <!-- Distance between the two camera lens centers -->
     <xacro:property name="camera_baseline" value="0.10"/>
+    <!-- Temporary approximate inertias for initial Gazebo testing -->
+    <xacro:macro name="simple_inertial" params="mass">
+        <inertial>
+            <origin xyz="0 0 0" rpy="0 0 0"/>
+            <mass value="${mass}"/>
+            <inertia
+                ixx="0.001"
+                ixy="0.0"
+                ixz="0.0"
+                iyy="0.001"
+                iyz="0.0"
+                izz="0.001"/>
+        </inertial>
+    </xacro:macro>
     <!-- ===================================================== -->
     <!-- MATERIALS                                             -->
@@ -42,4 +56,5 @@
     <!-- ===================================================== -->
     <link name="base_link">
+        <xacro:simple_inertial mass="1.0"/>
         <visual>
             <!--
@@ -65,4 +80,5 @@
     </joint>
     <link name="shoulder_link">
+        <xacro:simple_inertial mass="0.30"/>
         <visual>
             <origin xyz="0 0 0" rpy="0 0 0"/>
@@ -86,4 +102,5 @@
     </joint>
     <link name="forearm_link">
+        <xacro:simple_inertial mass="0.20"/>
         <visual>
             <origin xyz="0 0 -0.10597" rpy="0 0 0"/>
@@ -107,4 +124,5 @@
     </joint>
     <link name="elbow_link">
+        <xacro:simple_inertial mass="0.20"/>
         <visual>
             <origin xyz="-0.1778 0 -0.10597" rpy="0 0 0"/>
@@ -128,4 +146,5 @@
     </joint>
     <link name="wrist_link">
+        <xacro:simple_inertial mass="0.15"/>
         <visual>
             <origin xyz="-0.3302 0 -0.10597" rpy="0 0 0"/>
@@ -143,4 +162,5 @@
     </joint>
     <link name="end_effector_link">
+        <xacro:simple_inertial mass="0.15"/>
         <visual>
             <origin xyz="-0.3647 0 -0.10597" rpy="0 0 0"/>
@@ -163,4 +183,5 @@
     <!-- ===================================================== -->
     <link name="camera_stand_link">
+        <xacro:simple_inertial mass="0.20"/>
         <visual>
             <!--
@@ -189,4 +210,5 @@
     <!-- ===================================================== -->
     <link name="camera_mount_link">
+        <xacro:simple_inertial mass="0.10"/>
         <visual>
             <origin xyz="0 0 0" rpy="0 0 0"/>
@@ -216,4 +238,5 @@
     <!-- ===================================================== -->
     <link name="left_camera_link">
+        <xacro:simple_inertial mass="0.05"/>
         <visual>
             <origin xyz="0 0 0" rpy="0 0 0"/>
@@ -236,4 +259,5 @@
     <!-- ===================================================== -->
     <link name="right_camera_link">
+        <xacro:simple_inertial mass="0.05"/>
         <visual>
             <origin xyz="0 0 0" rpy="0 0 0"/>
@@ -277,3 +301,75 @@
             rpy="-1.5708 0 -1.5708"/>
     </joint>
+    <gazebo>
+        <static>true</static>
+    </gazebo>
+        <!-- ===================================================== -->
+    <!-- GAZEBO CAMERA SENSORS                                 -->
+    <!-- ===================================================== -->
+    <!-- Keep the camera links as separate Gazebo links -->
+    <gazebo reference="left_camera_joint">
+        <preserveFixedJoint>true</preserveFixedJoint>
+    </gazebo>
+    <gazebo reference="right_camera_joint">
+        <preserveFixedJoint>true</preserveFixedJoint>
+    </gazebo>
+    <!-- LEFT CAMERA SENSOR -->
+    <gazebo reference="left_camera_link">
+        <sensor name="left_camera_sensor" type="camera">
+            <always_on>true</always_on>
+            <update_rate>15</update_rate>
+            <visualize>true</visualize>
+            <!-- Gazebo image topic -->
+            <topic>/stereo/left/image_raw</topic>
+            <!-- Frame placed in ROS message headers -->
+            <gz_frame_id>left_camera_optical_frame</gz_frame_id>
+            <camera name="left_camera">
+                <camera_info_topic>
+                    /stereo/left/camera_info
+                </camera_info_topic>
+                <!-- Initial 60-degree horizontal field of view -->
+                <horizontal_fov>1.0472</horizontal_fov>
+                <image>
+                    <width>640</width>
+                    <height>480</height>
+                    <format>R8G8B8</format>
+                </image>
+                <clip>
+                    <near>0.05</near>
+                    <far>5.0</far>
+                </clip>
+            </camera>
+        </sensor>
+    </gazebo>
+    <!-- RIGHT CAMERA SENSOR -->
+    <gazebo reference="right_camera_link">
+        <sensor name="right_camera_sensor" type="camera">
+            <always_on>true</always_on>
+            <update_rate>15</update_rate>
+            <visualize>true</visualize>
+            <!-- Gazebo image topic -->
+            <topic>/stereo/right/image_raw</topic>
+            <!-- Frame placed in ROS message headers -->
+            <gz_frame_id>right_camera_optical_frame</gz_frame_id>
+            <camera name="right_camera">
+                <camera_info_topic>
+                    /stereo/right/camera_info
+                </camera_info_topic>
+                <horizontal_fov>1.0472</horizontal_fov>
+                <image>
+                    <width>640</width>
+                    <height>480</height>
+                    <format>R8G8B8</format>
+                </image>
+                <clip>
+                    <near>0.05</near>
+                    <far>5.0</far>
+                </clip>
+            </camera>
+        </sensor>
+    </gazebo>
+    <!-- Keep the whole model fixed during perception testing -->
+    <gazebo>
+        <static>true</static>
+    </gazebo>
 </robot>

Commit message: IK kinda working again

File: src/tomato_description/urdf/tomato_arm.urdf.xacro (robot description, xacro)
@@ -74,6 +74,7 @@
         <parent link="base_link"/>
         <child link="shoulder_link"/>
-        <!-- Arm orientation already matches the real robot -->
-        <origin xyz="0 0 0" rpy="0 0 0"/>
+        <!-- Physical joint_1 zero is rotated 180 degrees about base Z. -->
+        <!-- This rotates the shoulder and the entire descendant arm chain once. -->
+        <origin xyz="0 0 0" rpy="0 0 3.14159265359"/>
         <axis xyz="0 0 1"/>
         <limit effort="1.0" velocity="2.0"/>
@@ -92,7 +93,7 @@
     <joint name="joint_2" type="revolute">
         <parent link="shoulder_link"/>
-        <child link="forearm_link"/>
+        <child link="bicep_link"/>
         <origin xyz="0 0 0.10597" rpy="0 -1.5708 0"/>
-        <axis xyz="0 1 0"/>
+        <axis xyz="0 -1 0"/>
         <limit
             lower="-1.618"
@@ -101,5 +102,5 @@
             velocity="2.0"/>
     </joint>
-    <link name="forearm_link">
+    <link name="bicep_link">
         <xacro:simple_inertial mass="0.20"/>
         <visual>
@@ -107,5 +108,5 @@
             <geometry>
                 <mesh
-                    filename="package://tomato_description/meshes/forearm_link.stl"/>
+                    filename="package://tomato_description/meshes/bicep_link.stl"/>
             </geometry>
             <material name="color3"/>
@@ -113,8 +114,8 @@
     </link>
     <joint name="joint_3" type="revolute">
-        <parent link="forearm_link"/>
-        <child link="elbow_link"/>
+        <parent link="bicep_link"/>
+        <child link="forearm_link"/>
         <origin xyz="0.1778 0 0" rpy="0 0 0"/>
-        <axis xyz="0 1 0"/>
+        <axis xyz="0 -1 0"/>
         <limit
             lower="-1.825"
@@ -123,5 +124,5 @@
             velocity="2.0"/>
     </joint>
-    <link name="elbow_link">
+    <link name="forearm_link">
         <xacro:simple_inertial mass="0.20"/>
         <visual>
@@ -129,5 +130,5 @@
             <geometry>
                 <mesh
-                    filename="package://tomato_description/meshes/elbow_link.stl"/>
+                    filename="package://tomato_description/meshes/forearm_link.stl"/>
             </geometry>
             <material name="color4"/>
@@ -135,8 +136,8 @@
     </link>
     <joint name="joint_4" type="revolute">
-        <parent link="elbow_link"/>
+        <parent link="forearm_link"/>
         <child link="wrist_link"/>
         <origin xyz="0.1524 0 0" rpy="0 0 0"/>
-        <axis xyz="0 1 0"/>
+        <axis xyz="0 -1 0"/>
         <limit
             lower="-1.855"
@@ -162,11 +163,8 @@
     </joint>
     <link name="end_effector_link">
-        <xacro:simple_inertial mass="0.15"/>
         <visual>
             <origin xyz="-0.3647 0 -0.10597" rpy="0 0 0"/>
             <geometry>
-                <mesh
-                    filename="package://tomato_description/meshes/end_effector_link.stl"
-                    scale="0.001 0.001 0.001"/>
+                <mesh filename="package://tomato_description/meshes/end_effector_link.stl"/>
             </geometry>
             <material name="color5"/>
@@ -177,5 +175,5 @@
         <parent link="end_effector_link"/>
         <child link="tool_tip_link"/>
-        <origin xyz="0.124 0 0.04416" rpy="0 0 0"/>
+        <origin xyz="0.0925 -0.054675 0" rpy="0 0 0"/>
     </joint>
     <!-- ===================================================== -->
@@ -304,5 +302,5 @@
         <static>true</static>
     </gazebo>
-        <!-- ===================================================== -->
+    <!-- ===================================================== -->
     <!-- GAZEBO CAMERA SENSORS                                 -->
     <!-- ===================================================== -->
