Commit message: URDF changes again

File: src/tomato_description/urdf/tomato_arm.urdf.xacro (robot description, xacro)
@@ -5,5 +5,5 @@
     <!-- ===================================================== -->
     <!--
-        base_link convention:
+        Robot convention:
         +X = forward
         -X = backward
@@ -94,5 +94,5 @@
         <parent link="shoulder_link"/>
         <child link="bicep_link"/>
-        <origin xyz="0 0 0.10597" rpy="0 -1.5708 0"/>
+        <origin xyz="0 0 0.10897" rpy="0 -1.5708 0"/>
         <axis xyz="0 -1 0"/>
         <limit
@@ -105,5 +105,5 @@
         <xacro:simple_inertial mass="0.20"/>
         <visual>
-            <origin xyz="0 0 -0.10597" rpy="0 0 0"/>
+            <origin xyz="0 0 -0.10897" rpy="0 0 0"/>
             <geometry>
                 <mesh
@@ -127,5 +127,5 @@
         <xacro:simple_inertial mass="0.20"/>
         <visual>
-            <origin xyz="-0.1778 0 -0.10597" rpy="0 0 0"/>
+            <origin xyz="-0.1778 0 -0.10897" rpy="0 0 0"/>
             <geometry>
                 <mesh
@@ -149,5 +149,5 @@
         <xacro:simple_inertial mass="0.15"/>
         <visual>
-            <origin xyz="-0.3302 0 -0.10597" rpy="0 0 0"/>
+            <origin xyz="-0.3302 0 -0.10897" rpy="0 0 0"/>
             <geometry>
                 <mesh
@@ -164,5 +164,5 @@
     <link name="end_effector_link">
         <visual>
-            <origin xyz="-0.3647 0 -0.10597" rpy="0 0 0"/>
+            <origin xyz="-0.3647 0 -0.10897" rpy="0 0 0"/>
             <geometry>
                 <mesh filename="package://tomato_description/meshes/end_effector_link.stl"/>

Commit message: Kinda working again I cant rly tell ngl

File: src/tomato_description/urdf/tomato_arm.urdf.xacro (robot description, xacro)
@@ -5,5 +5,5 @@
     <!-- ===================================================== -->
     <!--
-        Robot convention:
+        base_link convention:
         +X = forward
         -X = backward
@@ -76,5 +76,5 @@
         <!-- Physical joint_1 zero is rotated 180 degrees about base Z. -->
         <!-- This rotates the shoulder and the entire descendant arm chain once. -->
-        <origin xyz="0 0 0" rpy="0 0 3.14159265359"/>
+        <origin xyz="0 0 0.06785" rpy="0 0 3.14159265359"/>
         <axis xyz="0 0 1"/>
         <limit effort="1.0" velocity="2.0"/>
@@ -83,5 +83,5 @@
         <xacro:simple_inertial mass="0.30"/>
         <visual>
-            <origin xyz="0 0 0" rpy="0 0 0"/>
+            <origin xyz="0 0 -0.06785" rpy="0 0 0"/>
             <geometry>
                 <mesh
@@ -94,5 +94,5 @@
         <parent link="shoulder_link"/>
         <child link="bicep_link"/>
-        <origin xyz="0 0 0.10897" rpy="0 -1.5708 0"/>
+        <origin xyz="0 0 0.04112" rpy="0 -1.5708 0"/>
         <axis xyz="0 -1 0"/>
         <limit
@@ -105,5 +105,5 @@
         <xacro:simple_inertial mass="0.20"/>
         <visual>
-            <origin xyz="0 0 -0.10897" rpy="0 0 0"/>
+            <origin xyz="0 0 -0.10597" rpy="0 0 0"/>
             <geometry>
                 <mesh
